File: STM32F4_REV2/STM32F4_REV2.kicad_pcb (KiCad board)
At the start: 4 copper layers, 49.2 x 47.8 mm, 50 parts, among them IC1 MP2359DJ-LF-Z, J1 Screw_Terminal_01x02, J2 SWD, J3 Conn_01x04, J4 Conn_01x04, J5 USB_B_Micro, Q1 AO3401A, SW1 SW_SPDT, U1 STM32F405RGT6, U2 USBLC6-2SC6, Y1 16MHz

Commit message: Uploading the PCB files
Parts:
- added Housing: ToolingHole_1.152mm, MountingHole:ToolingHole_1.152mm, F.Cu at (157.5, 79.8)
- added Housing: ToolingHole_1.152mm, MountingHole:ToolingHole_1.152mm, F.Cu at (133.2, 118.8)
- added Housing: ToolingHole_1.152mm, MountingHole:ToolingHole_1.152mm, F.Cu at (133.2, 79.8)
- added Housing: ToolingHole_1.152mm, MountingHole:ToolingHole_1.152mm, F.Cu at (157.5, 118.8)
- moved D2 30.8 mm to (157.6, 84.0), turned to 0 degrees
- moved R4 26.1 mm to (157.7, 85.9)
- moved R1 8.03 mm to (128.7, 89.7)
- moved R11 1.90 mm to (140.0, 88.1)
- moved C11 0.95 mm to (127.3, 100.0)
- moved R2 0.94 mm to (131.8, 98.0), turned to -90 degrees
- moved C1 0.92 mm to (148.6, 95.3), turned to 0 degrees
- moved C16 0.91 mm to (153.9, 115.3), turned to 180 degrees
- moved C17 0.91 mm to (148.8, 115.3)
- moved C6 0.78 mm to (137.0, 107.2)
- moved C2 0.78 mm to (142.8, 107.2)
- moved D3 0.78 mm to (149.5, 104.5), turned to 0 degrees
- moved R12 0.72 mm to (139.0, 90.5)
- moved C4 0.71 mm to (136.7, 90.5)
- moved D4 0.41 mm to (156.5, 98.1)
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- renumbered D1 to STATUS
Connections:
- net IC1_GND renamed GND
- U1 pad 44: USB_DM -> USB_D-
- U1 pad 45: USB_DP -> USB_D+
- U2 pad 1: USB_DM -> USB_D+
- U2 pad 3: USB_CONN_D- -> USB_D-
- U2 pad 4: USB_CONN_D+ -> USB_CONN_D-
- U2 pad 6: USB_DP -> USB_CONN_D+
Routing:
- net GND: track 0.00 -> 122.5 mm, vias 0 -> 53
- net +3.3V: track 0.00 -> 54.6 mm, vias 0 -> 29
- net SWO: track 0.00 -> 31.5 mm, vias 0 -> 2
- net NRST: track 0.00 -> 29.4 mm, vias 0 -> 2
- net IC1_SW: track 0.00 -> 17.6 mm
- net SWCLK: track 0.00 -> 15.0 mm
- net I2C1_SCL: track 0.00 -> 14.7 mm
- net UART3_TX: track 0.00 -> 14.3 mm
- net I2C1_SDA: track 0.00 -> 14.2 mm
- net SWDIO: track 0.00 -> 14.1 mm
- net UART3_RX: track 0.00 -> 13.6 mm
- net Net-(C11-Pad1): track 0.00 -> 12.5 mm, vias 0 -> 2
- net BOOT0: track 0.00 -> 11.8 mm
- net USB_D+: track 0.00 -> 11.8 mm
- net USB_D-: track 0.00 -> 11.2 mm
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- added copper zone on In2.Cu, net +3.3V
- added copper zone on In1.Cu, net GND
Other:
- board text added: "+"
- board text added: "-"
- board text added: "<"
- board text added: "Quanttronix"
- board text added: "Qx"
- board text added: "RUN"
- board text added: "STM32F4 Project 1 Board | vSEP 2026"

Commit message: Uploading the PCB files kanboard #7406
Parts:
- added C17: 100n, Capacitor_SMD:C_0402_1005Metric, F.Cu at (123.0, 102.0)
- added J6: Conn_01x04, Connector_Molex:Molex_PicoBlade_53048-0410_1x04_P1.25mm_Horizontal, F.Cu at (108.9, 122.0)
- added J7: Conn_01x04, Connector_Molex:Molex_PicoBlade_53048-0410_1x04_P1.25mm_Horizontal, F.Cu at (147.9, 76.8)
- added R5: 10k, Resistor_SMD:R_0603_1608Metric, F.Cu at (128.2, 102.8)
- added SW2: SW_Push, Button_Switch_THT:SW_PUSH_6mm_H5mm, F.Cu at (129.2, 109.5)
- added TP1: TestPoint, Connector_PinHeader_2.54mm:PinHeader_1x01_P2.54mm_Vertical, F.Cu at (107.0, 95.5)
- added TP2: TestPoint, Connector_PinHeader_2.54mm:PinHeader_1x01_P2.54mm_Vertical, F.Cu at (107.0, 100.1)
- added TP3: TestPoint, Connector_PinHeader_2.54mm:PinHeader_1x01_P2.54mm_Vertical, F.Cu at (107.0, 104.7)
- added TP4: TestPoint, Connector_PinHeader_2.54mm:PinHeader_1x01_P2.54mm_Vertical, F.Cu at (106.2, 109.2)
- added TP5: TestPoint, Connector_PinHeader_2.54mm:PinHeader_1x01_P2.54mm_Vertical, F.Cu at (111.2, 115.8)
- moved J2 1.43 mm to (149.9, 87.5)
- moved R3 1.03 mm to (132.5, 107.2)
- moved C2 0.90 mm to (143.2, 108.0), turned to -90 degrees
- renumbered C15 to C14, C16 to C15, C17 to C16, STATUS to STATUS1
Connections:
- net +3.3V renamed VBAT_TP
- net +3.3VA renamed VDDA_TP
- J2 pad 10: NRST -> unconnected-(J2-Pin_10-Pad10)
- U1 pad 17: SWO -> unconnected-(U1-PA3-Pad17)
- U1 pad 55: unconnected-(U1-PB3-Pad55) -> SWO
Routing:
- net SWO: track 31.5 -> 0.00 mm, vias 2 -> 0
- net SWCLK: track 15.0 -> 0.00 mm
- net SWDIO: track 14.1 -> 0.00 mm
- net GND: track 122.5 -> 130.8 mm, vias 53 -> 58
- net NRST: track 29.4 -> 24.0 mm
- net VBAT_TP: track 54.6 -> 55.8 mm, vias 29 -> 30
- net Net-(STATUS1-K): track 2.02 -> 3.04 mm
- net Net-(U1-VCAP_1): track 3.37 -> 2.84 mm
