File: STM32F4_REV2/STM32F4_REV2.kicad_pcb (KiCad board)
At the start: 4 copper layers, 49.2 x 47.8 mm, 66 parts, among them IC1 MP2359DJ-LF-Z, J1 Screw_Terminal_01x02, J2 SWD, J3 Conn_01x04, J4 Conn_01x04, J5 USB_B_Micro, J6 Conn_01x04, J7 Conn_01x04, J8 Conn_01x02, Q1 AO3401A, SW1 SW_SPDT, SW2 SW_Push, U1 STM32F405RGT6, U2 USBLC6-2SC6, Y1 16MHz

Commit message: Uploading the PCB files kanboard #7406
Parts:
- removed L1: 39n, Inductor_SMD:L_0805_2012Metric
- added FB2: BLM21PG221SN1D, DownloadedLib:BEADC2012X105N, F.Cu at (127.6, 101.1)
- added FID1: Fiducial, Fiducial:Fiducial_1mm_Mask2mm, F.Cu at (160.1, 75.5)
- added FID2: Fiducial, Fiducial:Fiducial_1mm_Mask2mm, F.Cu at (130.7, 75.5)
- added FID3: Fiducial, Fiducial:Fiducial_1mm_Mask2mm, F.Cu at (130.7, 120.0)
- added FID4: Fiducial, Fiducial:Fiducial_1mm_Mask2mm, F.Cu at (160.1, 120.0)
- moved R10 5.29 mm to (158.1, 115.2), turned to 180 degrees
- moved C12 4.11 mm to (132.0, 95.4), turned to 90 degrees
- moved R8 3.31 mm to (155.2, 114.2), turned to 90 degrees
- moved C8 2.67 mm to (148.7, 92.7)
- moved R7 2.62 mm to (161.2, 109.9)
- moved C15 2.28 mm to (151.6, 115.4)
- moved C11 2.23 mm to (126.0, 98.3), turned to 180 degrees
- moved C16 2.07 mm to (146.7, 115.4)
- moved C5 1.57 mm to (132.7, 92.6), turned to 180 degrees
- moved R6 1.56 mm to (157.7, 109.9), turned to 0 degrees
- moved Y1 1.52 mm to (127.3, 95.3)
- moved R2 0.99 mm to (131.3, 98.2), turned to 180 degrees
- moved TP1 0.92 mm to (131.8, 105.2)
- moved R3 0.90 mm to (132.7, 109.7)
- moved D1 0.90 mm to (132.7, 107.6)
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Routing:
- net GND: track 0.00 -> 82.7 mm, vias 0 -> 28
- net +3.3V: track 2.87 -> 59.6 mm, vias 2 -> 19
- net NRST: track 0.00 -> 30.9 mm, vias 0 -> 2
- net RGB7_TP: track 0.00 -> 26.7 mm, vias 0 -> 2
- net SWO: track 0.00 -> 24.1 mm
- net I2C1_SCL: track 0.00 -> 24.0 mm
- net UART3_RX: track 0.00 -> 22.3 mm
- net I2C1_SDA: track 0.00 -> 21.5 mm
- net UART3_TX: track 0.00 -> 21.3 mm
- net RGB6_TP: track 0.00 -> 20.1 mm, vias 0 -> 2
- net RGB5_TP: track 0.00 -> 20.0 mm, vias 0 -> 2
- net SWCLK: track 0.00 -> 18.5 mm
- net GPIO_TEST: track 0.00 -> 17.0 mm
- net IC1_SW: track 0.00 -> 17.0 mm
- net SWDIO: track 0.00 -> 15.4 mm
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Other:
- board text added: "12v"
- board text added: "3v3"
- board text added: "GND"
- board text added: "GPIO_TP"
- board text added: "I2C_TP"
- board text added: "LED"
- board text added: "Moustafa Mekawy"
- board text added: "NRST"
- board text added: "PA4"
- board text added: "QX v1.0"
- board text added: "RX"
- board text added: "SCL"
- board text added: "SDA"
- board text added: "SN: 25445216648"
- board text added: "SW"
- board text added: "TX"
- board text added: "UART_TP"
- board text added: "USB"
- board text added: "VATP"
- board text added: "Vdd"
- board text added: "X"
- board text removed: "STM32F4 Project 1 Board | vSEP 2026"

Commit message: Modified
Parts:
- D3, D4: value B230 -> B230AF-13; footprint Diode_SMD:D_SOD-123 -> DownloadedLib:SODFL5226X110N
- moved F1 0.89 mm to (152.2, 98.6)
- moved FB1 0.40 mm to (152.5, 103.5)
- moved D3 0.22 mm to (149.5, 103.3)
- moved D4 0.22 mm to (156.3, 98.0)
- moved C15 0.20 mm to (151.6, 115.6)
- moved C16 0.20 mm to (146.7, 115.6)
- turned C14 to 180 degrees
Connections:
- net IC1_EN renamed Net-(IC1-EN)
- net IC1_FB renamed Net-(IC1-FB)
- net IC1_IN renamed Net-(IC1-IN)
- C14 pad 1: IC1_BST -> Net-(D3-K)
- C14 pad 2: IC1_SW -> Net-(IC1-BST)
- D3 pad 1: IC1_SW -> Net-(D3-K)
- IC1 pad 1: IC1_BST -> Net-(IC1-BST)
- IC1 pad 6: IC1_SW -> Net-(D3-K)
- L2 pad 1: IC1_SW -> Net-(D3-K)
- Y1 pad 2: GND -> Net-(Y1-G-Pad2)
- Y1 pad 4: GND -> Net-(Y1-G-Pad2)
Routing:
- net IC1_SW: track 17.0 -> 0.00 mm
- net Net-(D3-K): track 0.00 -> 16.1 mm
- net +3.3V: track 59.6 -> 57.3 mm, vias 19 -> 18
- net Net-(IC1-BST): track 0.00 -> 2.24 mm
- net IC1_BST: track 2.24 -> 0.00 mm
- net Net-(Y1-G-Pad2): track 0.00 -> 1.73 mm
- net GND: track 82.7 -> 81.3 mm
- net Net-(F1-Pad2): track 3.52 -> 4.65 mm
- net UART3_TX: track 21.3 -> 22.3 mm
- net +5V: track 13.6 -> 12.7 mm
- net Net-(IC1-IN): track 10.6 -> 10.0 mm

Commit message: Fixing most the bugs and following the checklist
Parts:
- removed RGB1: 150080M153000, DownloadedLib:150080M153000
- added LED1: UHD111A-FKA-C3K23E1L3VG5ZB3Z3, M_Design_Lib:UHD111AFKAC3K23E1L3VG5ZB3Z3, F.Cu at (138.2, 114.5)
- D3, D4: footprint DownloadedLib:SODFL5226X110N -> M_Design_Lib:SODFL5226X110N
- FB1: value 600 @ 600 MHz -> 600 @ 100 MHz
- FB2: footprint DownloadedLib:BEADC2012X105N -> M_Design_Lib:BEADC2012X105N
- IC1: footprint DownloadedLib:MP2359DJ-LF-Z -> M_Design_Lib:MP2359DJ-LF-Z
- J5: footprint DownloadedLib:101181930001LF -> M_Design_Lib:101181930001LF
- R11, R12: value 4k7 -> 3k3
- R13, R15: value 1k -> 220
- R14: value 1k -> 330
- R7: value 68k -> 100k
- Z1: footprint DownloadedLib:SOD2512X110N -> M_Design_Lib:SOD2512X110N
- moved TP2 30.0 mm to (134.0, 84.0)
- moved R15 27.8 mm to (138.0, 110.7), turned to 90 degrees
- moved R14 26.1 mm to (136.0, 110.7), turned to 90 degrees
- moved R13 23.8 mm to (140.0, 110.7), turned to -90 degrees
- moved TP1 21.2 mm to (131.0, 84.0)
- moved TP4 20.9 mm to (137.0, 84.0)
- moved L1 19.7 mm to (167.2, 111.6), turned to 0 degrees
- moved TP3 19.3 mm to (134.0, 80.2)
- moved J7 14.0 mm to (147.7, 77.4), turned to 90 degrees
- moved D3 6.43 mm to (151.2, 109.5), turned to -90 degrees
- moved Q1 6.10 mm to (160.5, 99.8), turned to 0 degrees
- moved J2 5.34 mm to (149.2, 84.5), turned to -90 degrees
- moved IC1 5.17 mm to (157.5, 109.5)
- moved D4 4.81 mm to (159.6, 94.5), turned to 0 degrees
- moved R6 4.74 mm to (161.6, 107.2)
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- renumbered L2 to L1
Connections:
- R13 pad 1: Net-(RGB1-K_RED) -> RGB7_TP
- R13 pad 2: RGB5_TP -> Net-(LED1-CATHODE_BLUE)
- R14 pad 2: RGB6_TP -> RGB5_TP
- R15 pad 2: RGB7_TP -> RGB6_TP
- Z1 pad 1: +12V -> Net-(D4-K)
Routing:
- net +3.3VA: track 10.5 -> 34.2 mm, vias 0 -> 2
- net RGB7_TP: track 26.7 -> 5.67 mm, vias 2 -> 0
- net GND: track 81.3 -> 62.8 mm, vias 28 -> 25
- net NRST: track 30.9 -> 45.2 mm, vias 2 -> 3
- net RGB6_TP: track 20.1 -> 6.30 mm, vias 2 -> 0
- net RGB5_TP: track 20.0 -> 6.92 mm, vias 2 -> 0
- net SWO: track 24.1 -> 11.7 mm
- net Net-(D4-K): track 6.48 -> 18.2 mm
- net SWCLK: track 18.5 -> 9.99 mm
- net I2C1_SDA: track 21.5 -> 28.1 mm
- net +3.3V: track 57.3 -> 50.7 mm, vias 18 -> 16
- net Net-(IC1-EN): track 11.3 -> 6.26 mm
- net UART3_RX: track 22.3 -> 27.2 mm
- net USB_D-: track 10.5 -> 14.6 mm
- net Net-(LED1-CATHODE_BLUE): track 0.00 -> 4.05 mm
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Other:
- board size 49.2 x 47.8 mm -> 50.8 x 50.7 mm
- board text added: "Power Circuit"
- board text added: "RGB"
- board text added: "TP Area"
- board text added: "▲"

Commit message: Modified
Parts:
- C11, C12: value 12p -> 18p
- moved C16 0.58 mm to (151.3, 115.5)
- moved C15 0.58 mm to (153.9, 115.5)
- moved C17 0.10 mm to (122.5, 102.4)
- moved R5 0.10 mm to (124.7, 102.4)
- moved Q1 0.06 mm to (160.5, 99.7)
- moved U2 0.06 mm to (159.8, 90.8)
- moved Z1 0.06 mm to (155.4, 101.3)
- moved J2 0.06 mm to (149.2, 84.4)
Connections:
- Y1 pad 2: Net-(Y1-G-Pad2) -> GND
- Y1 pad 4: Net-(Y1-G-Pad2) -> GND
Routing:
- net GND: track 62.8 -> 66.9 mm, vias 25 -> 26
- net Net-(Y1-G-Pad2): track 2.90 -> 0.00 mm
- net NRST: track 45.2 -> 47.9 mm
- net I2C1_SCL: track 21.4 -> 22.3 mm
- net Net-(IC1-FB): track 6.51 -> 7.39 mm
- net Net-(IC1-IN): track 11.0 -> 11.7 mm
Other:
- board text added: "TPArea"
- board text removed: "TP Area"

Commit message: Modified'
Parts:
- moved J1 0.10 mm to (166.4, 102.6)
Changed lines of the file:
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@@
 	(footprint "TerminalBlock_Phoenix:TerminalBlock_Phoenix_PT-1,5-2-3.5-H_1x02_P3.50mm_Horizontal"
 		(layer "F.Cu")
-		(at 166.5 102.6 90)
+		(at 166.4 102.6 90)
 		(descr "Terminal Block Phoenix PT-1,5-2-3.5-H, 2 pins, pitch 3.5mm, size 7x7.6mm, drill diameter 1.2mm, pad diameter 2.4mm, ")
 		(tags "THT Terminal Block Phoenix PT-1,5-2-3.5-H pitch 3.5mm size 7x7.6mm drill 1.2mm pad 2.4mm")
@@
 	)
 	(segment
-		(start 161.5375 99.8)
-		(end 161.4375 99.7)
+		(start 164.325 102.6)
+		(end 161.5375 99.8125)
 		(width 0.5)
 		(layer "F.Cu")
@@
 	)
 	(segment
-		(start 166.5 102.6)
+		(start 166.4 102.6)
 		(end 164.325 102.6)
 		(width 0.5)
@@
 	)
 	(segment
-		(start 164.325 102.6)
-		(end 161.5375 99.8125)
+		(start 161.5375 99.8)
+		(end 161.4375 99.7)
 		(width 0.5)
 		(layer "F.Cu")
