File: STM32F4_REV2/STM32F4_REV2.kicad_sch (KiCad schematic)
At the start: 66 parts, among them IC1 MP2359DJ-LF-Z, J1 Screw_Terminal_01x02, J2 SWD, J3 Conn_01x04, J4 Conn_01x04, J5 USB_B_Micro, J6 Conn_01x04, J7 Conn_01x04, J8 Conn_01x02, Q1 AO3401A, SW1 SW_SPDT, SW2 SW_Push, U1 STM32F405RGT6, U2 USBLC6-2SC6, Y1 16MHz

Commit message: Uploading the PCB files kanboard #7406
Parts:
- removed L1: 39n, Inductor_SMD:L_0805_2012Metric, symbol Device:L_Small
- added FB2: BLM21PG221SN1D, BEADC2012X105N, symbol DownloadedLib:BLM21PG221SN1D
- added FID1, FID2, FID3, FID4: Fiducial, Fiducial:Fiducial_1mm_Mask2mm, symbol Mechanical:Fiducial
Connections:
- net +3.3V: now also FB2.1
- net +3.3VA: now also FB2.2

Commit message: Modified
Parts:
- removed D3, D4: B230, Diode_SMD:D_SOD-123, symbol Diode:B230
- added D3, D4: B230AF-13, DownloadedLib:SODFL5226X110N, symbol DownloadedLib:B230AF-13
- C1, C2: #DigiKey (none) -> 399-C0805C225J4RECTUCT-ND; #MFR (none) -> C0805C225J4RECTU
- C10, C14: #DigiKey (none) -> 399-17422-1-ND; #MFR (none) -> C0805C103J5RACTU
- C11, C12: #DigiKey (none) -> 399-17427-1-ND; #MFR (none) -> C0805C120J3GACTU
- C13, C15, C16: #DigiKey (none) -> 4988-NMC1206X5R106K25TRPLPFCT-ND; #MFR (none) -> NMC1206X5R106K25TRPLPF
- C17, C4, C5, C6, C7, C8: #DigiKey (none) -> 13-CC0805KPX7R7BB104CT-ND; #MFR (none) -> CC0805KPX7R7BB104
- C3: #DigiKey (none) -> C0805C225J4RECTU; #MFR (none) -> TMK212AB7475KG-T
- C9: #DigiKey (none) -> 311-1365-1-ND; #MFR (none) -> CC0805KKX7R7BB105
- D1: #DigiKey (none) -> 1516-QBLP631-IB5-2897CT-ND; #MFR (none) -> QBLP631-IB5-2897
- D2: #DigiKey (none) -> 754-1097-1-ND; #MFR (none) -> APHCM2012SURCK-F01
- F1: #DigiKey (none) -> 283-CC12H250MA-TRCT-ND; #MFR (none) -> CC12H250MA-TR
- FB1: value 600 @ 600 MHz -> 600 @ 100 MHz; #DigiKey (none) -> 445-MPZ2012S601AT000CT-ND; #MFR (none) -> MPZ2012S601AT000
- FB2: footprint BEADC2012X105N -> DownloadedLib:BEADC2012X105N; #DigiKey (none) -> 490-1054-1-ND; #MFR (none) -> BLM21PG221SN1D
- IC1: #DigiKey (none) -> 1589-1889-2-ND; #MFR (none) -> MP2359DJ-LF-Z
- J1: #DigiKey (none) -> Phoenix Contact 1984617; #MFR (none) -> 1984617
- J2: #DigiKey (none) -> SAM8799-ND; #MFR (none) -> FTSH-105-01-L-DV-K
- J3, J4: #DigiKey (none) -> WM1744-ND; #MFR (none) -> 0530480410
- J5: #DigiKey (none) -> 609-4616-1-ND; #MFR (none) -> 10118193-0001LF
- J6, J7, J8: #DigiKey (none) -> WM23244-ND; #MFR (none) -> 0423751247
- L1: renamed from L2; #DigiKey (none) -> 3442-MWSA0518S-100MTCT-ND; #MFR (none) -> MWSA0518S-100MT
- Q1: #DigiKey (none) -> 785-1001-1-ND; #MFR (none) -> AO3401A
- R1, R16, R5: #DigiKey (none) -> 738-RNCA0805BTE10K0CT-ND; #MFR (none) -> RNCA0805BTE10K0
- R10: #DigiKey (none) -> A130470CT-ND; #MFR (none) -> CRGP0805F270R
- R11, R12: #DigiKey (none) -> A129757CT-ND; #MFR (none) -> CRGCQ0805F4K7
- R13, R14, R15, R3, R4: #DigiKey (none) -> P123793CT-ND; #MFR (none) -> ERA-6AED102V
- R2: #DigiKey (none) -> P123850CT-ND; #MFR (none) -> ERA-6AED470V
- R6: #DigiKey (none) -> 13-RP0805BRD07100KLCT-ND; #MFR (none) -> RP0805BRD07100KL
- R7: value 68k -> 100k; #DigiKey (none) -> 13-RP0805BRD07100KLCT-ND; #MFR (none) -> RP0805BRD07100KL
- R8: #DigiKey (none) -> 1727-8643-1-ND; #MFR (none) -> 2N7002NXAKR
- R9: #DigiKey (none) -> P123809CT-ND; #MFR (none) -> ERA-6AED153V
- SW1: #DigiKey (none) -> 401-2016-1-ND; #MFR (none) -> PCM12SMTR
- SW2: #DigiKey (none) -> 2449-CT1102P5.0F100-ND; #MFR (none) -> CT1102P5.0F100
- U1: #DigiKey (none) -> 497-11767-ND; #MFR (none) -> STM32F405RGT6
- U2: #DigiKey (none) -> 497-5235-1-ND; #MFR (none) -> USBLC6-2SC6
- Y1: #DigiKey (none) -> 1908-1275-1-ND; #MFR (none) -> Q 16,0-JXS32-12-10/15-T1-WA-LF
- Z1: #DigiKey (none) -> 1727-BZX384-C8V2,115CT-ND; #MFR (none) -> BZX384-C8V2,115
Connections:
- net +12V: no longer Z1.1 (K)
- net +5V: now also D4.2 (A)
- net GND: now also D3.2 (A); no longer Y1.2 (G), Y1.4 (G)
- net at F1.1, Q1.2 (S): now also Z1.1 (K), D4.1 (K)
- net IC1_BST: no longer names the net of C14.1
- net IC1_BST: now also IC1.6 (SW), L1.1, D3.1 (K); no longer IC1.1 (BST)
- net IC1_EN: no longer names the net of IC1.4 (EN), R6.2, R7.1
- net IC1_FB: no longer names the net of IC1.3 (FB), R8.2, R9.1
- net IC1_IN: no longer names the net of C13.1, FB1.2, IC1.5 (IN), R6.1
- removed net IC1_SW: C14.2, IC1.6 (SW), L1.1
- new net: C14.2, IC1.1 (BST)
- new net: Y1.2 (G), Y1.4 (G)
Other:
- note added: "C = 2 * ( C + C )"
- note added: "Decoupling Caps Based on Datasheet"
- note added: "From Checklist"
- note added: "Initially RExt = 1 / (2 π F CL2)"
- note added: "It should be 20uF Phil's lab"
- note added: "L"
- note added: "Limit the drive level provided by the STM32 to protect the Crystal"
- note added: "PMOS Protection"
- note added: "Polarity Protection"
- note added: "Reference Circuit"
- note added: "Same Ratio as Suggested in the DataSheet"
- note added: "Within range 1-10 uH 4.7uH Recommended"
- note added: "load"
- note added: "stray"
- moved on the sheet: C10, C11, C12, C13, C14, C15, C16, C17, C9, D1, D2, F1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

Commit message: Fixing most the bugs and following the checklist
Parts:
- removed RGB1: 150080M153000, DownloadedLib:150080M153000, symbol DownloadedLib:150080M153000
- added LED1: UHD111A-FKA-C3K23E1L3VG5ZB3Z3, M_Design_Lib:UHD111AFKAC3K23E1L3VG5ZB3Z3, symbol M_Design_Lib:UHD111A-FKA-C3K23E1L3VG5ZB3Z3
- D3, D4: footprint DownloadedLib:SODFL5226X110N -> M_Design_Lib:SODFL5226X110N
- FB2: footprint DownloadedLib:BEADC2012X105N -> M_Design_Lib:BEADC2012X105N
- IC1: footprint DownloadedLib:MP2359DJ-LF-Z -> M_Design_Lib:MP2359DJ-LF-Z
- J5: footprint DownloadedLib:101181930001LF -> M_Design_Lib:101181930001LF
- R11, R12: value 4k7 -> 3k3; #DigiKey A129757CT-ND -> A129755CT-ND; #MFR CRGCQ0805F4K7 -> CRGCQ0805F3K3
- R13, R15: value 1k -> 220; #DigiKey P123793CT-ND -> A129741CT-ND; #MFR ERA-6AED102V -> CRGCQ0805F220R
- R14: value 1k -> 330; #DigiKey P123793CT-ND -> 273-KDV08FR330ETCT-ND; #MFR ERA-6AED102V -> KDV08FR330ET
- Z1: footprint DownloadedLib:SOD2512X110N -> M_Design_Lib:SOD2512X110N
Connections:
- net +3.3V: now also LED1.4 (COMMON_ANODE)
- net RGB5_TP: now also R14.2; no longer R13.2
- net RGB6_TP: now also R15.2; no longer R14.2
- net RGB7_TP: now also R13.1; no longer R15.2
- net at R14.1: now also LED1.3 (CATHODE_RED)
- net at R15.1: now also LED1.2 (CATHODE_GREEN)
- new net: LED1.1 (CATHODE_BLUE), R13.2
Other:
- note added: "@3mA If 10mA Imax 30mA"
- note added: "@5mA If 10mA Imax 30mA"
- note added: "Default High"
- note added: "I = 0.6 mA"
- note added: "If = 10 mA"
- note added: "If = 4.54 ~ 0.91 mA"
- note added: "If = 4.8 ~ 3 mA"
- note added: "Reference Device"
- note added: "This circuit values are made based on this sensor"
- note added: "Vf = 1.7 ~ 2.3v"
- note added: "Vf = 2.7v"
- note added: "Vf = 3.1 ~ 2.3v"
- moved on the sheet: C13, C14, C15, C16, D2, D3, D4, F1, FB1, FID1, FID2, FID3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

Commit message: Modified
Parts:
- C11, C12: value 12p -> 18p; #DigiKey 399-17427-1-ND -> 399-C0805C180J5GACTUCT-ND; #MFR C0805C120J3GACTU -> C0805C180J5GACTU
Connections:
- net GND: now also Y1.2 (G), Y1.4 (G)
Other:
- note added: "3v3 Indicator"
- note added: "C = 2 * ( C - C )"
- note added: "It should be 100k ohm between 5&4 but the extra 100k is make sure we are <6v"
- note removed: "C = 2 * ( C + C )"
- moved on the sheet: C11, C12, C17, D1, D2, FID1, FID2, FID3, FID4, H1, H2, H3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
