File: STM32F4_REV2/_restore_backup_2026-10-05T14-53-29-578/STM32F4_REV2.kicad_pcb (KiCad board)
At the start: 4 copper layers, 49.2 x 47.8 mm, 66 parts, among them IC1 MP2359DJ-LF-Z, J1 Screw_Terminal_01x02, J2 SWD, J3 Conn_01x04, J4 Conn_01x04, J5 USB_B_Micro, J6 Conn_01x04, J7 Conn_01x04, J8 Conn_01x02, Q1 AO3401A, SW1 SW_SPDT, SW2 SW_Push, U1 STM32F405RGT6, U2 USBLC6-2SC6, Y1 16MHz

Commit message: Uploading the PCB files kanboard #7406
Parts:
- added TP5: TestPoint, Connector_PinHeader_2.54mm:PinHeader_1x01_P2.54mm_Vertical, F.Cu at (111.2, 115.8)
- C1, C14, C2, C3: footprint Capacitor_SMD:C_0805_2012Metric -> Capacitor_SMD:C_0603_1608Metric
- C10, C11, C12, C17, C4, C5, C6, C7, C8, C9: footprint Capacitor_SMD:C_0805_2012Metric -> Capacitor_SMD:C_0402_1005Metric
- D2: footprint LED_SMD:LED_0805_2012Metric -> LED_SMD:LED_0603_1608Metric
- F1: value 250 mA -> 250mA
- L1: footprint Inductor_SMD:L_0805_2012Metric -> Inductor_SMD:L_0402_1005Metric
- R1, R11, R12, R2: footprint Resistor_SMD:R_0805_2012Metric -> Resistor_SMD:R_0402_1005Metric
- R10, R13, R14, R15, R16, R3, R4, R5, R6, R7, R8, R9: footprint Resistor_SMD:R_0805_2012Metric -> Resistor_SMD:R_0603_1608Metric
- STATUS1: renamed from D1; footprint LED_SMD:LED_0805_2012Metric -> LED_SMD:LED_0603_1608Metric
- moved R16 59.9 mm to (99.6, 92.4), turned to 0 degrees
- moved R13 46.8 mm to (99.6, 84.9)
- moved R15 43.1 mm to (99.6, 89.9), turned to 0 degrees
- moved R14 42.7 mm to (99.6, 87.4)
- moved TP2 38.1 mm to (107.0, 100.1)
- moved RGB1 30.5 mm to (134.2, 112.1), turned to 180 degrees
- moved TP1 26.4 mm to (107.0, 95.5)
- moved TP4 19.3 mm to (106.2, 109.2)
- moved TP3 17.8 mm to (107.0, 104.7)
- moved J7 12.2 mm to (145.7, 76.2), turned to 90 degrees
- moved Z1 5.31 mm to (159.3, 98.5), turned to 0 degrees
- moved C11 4.43 mm to (127.3, 100.0), turned to 0 degrees
- moved C3 3.93 mm to (132.2, 94.0), turned to 90 degrees
- moved J8 3.73 mm to (133.5, 120.5)
- moved R11 2.78 mm to (140.0, 88.1), turned to 0 degrees
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Connections:
- J5 pad MP1: (no net) -> unconnected-(J5-Shield-PadMP1)
Routing:
- net GND: track 0.00 -> 111.3 mm, vias 0 -> 53
- net +3.3V: track 2.87 -> 50.1 mm, vias 2 -> 26
- net NRST: track 0.00 -> 24.0 mm, vias 0 -> 2
- net IC1_SW: track 0.00 -> 17.6 mm
- net I2C1_SCL: track 0.00 -> 14.5 mm
- net UART3_TX: track 0.00 -> 14.3 mm
- net I2C1_SDA: track 0.00 -> 14.2 mm
- net UART3_RX: track 0.00 -> 13.6 mm
- net Net-(C11-Pad1): track 0.00 -> 12.5 mm, vias 0 -> 2
- net BOOT0: track 0.00 -> 11.8 mm
- net USB_D+: track 0.00 -> 11.8 mm
- net USB_D-: track 0.00 -> 11.2 mm
- net +5V: track 0.00 -> 10.6 mm
- net IC1_IN: track 0.00 -> 9.91 mm
- net IC1_FB: track 0.00 -> 9.00 mm
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