File: STM32F4_REV2/_restore_backup_2026-10-05T14-53-29-578/STM32F4_REV2.kicad_sch (KiCad schematic)
At the start: 66 parts, among them IC1 MP2359DJ-LF-Z, J1 Screw_Terminal_01x02, J2 SWD, J3 Conn_01x04, J4 Conn_01x04, J5 USB_B_Micro, J6 Conn_01x04, J7 Conn_01x04, J8 Conn_01x02, Q1 AO3401A, SW1 SW_SPDT, SW2 SW_Push, U1 STM32F405RGT6, U2 USBLC6-2SC6, Y1 16MHz

Commit message: Uploading the PCB files kanboard #7406
Parts:
- F1: value 250 mA -> 250mA
Changed lines of the file:
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@@
 			)
 		)
-		(property "Value" "250 mA"
+		(property "Value" "250mA"
 			(at 73.66 34.798 90)
 			(show_name no)
